File: Balanced Polarimeter/Balanced Polarimeter.kicad_sch (KiCad schematic)
At the start: 23 parts, among them IC1 OP27, J1 73100-0105, J2 Conn_01x03_Pin, J3 Conn_01x02_Pin, J5 Conn_01x02_Pin, Q1 MMPQ3904, Q2 MMPQ3904, U1 ADA4898-1YRDZ, U2 ADA4898-1YRDZ

Commit message: Revised Wiring
Connections:
- net +5V: now also Q1.3 (COLLECTOR_#2_1), Q1.4 (COLLECTOR_#2_2), Q2.3 (COLLECTOR_#2_1), Q2.4 (COLLECTOR_#2_2); no longer D1.3 (A), D2.3 (A)
- net -5V: now also D1.1 (K), D2.1 (K)
- net GND: now also U1.3 (+), U2.3 (+)
- net at Q2.1 (COLLECTOR_DYE_#1), Q2.13 (BASE_#2), Q2.2 (COLLECTOR_#1): now also D1.3 (A)
- net at Q2.5 (COLLECTOR_#3_1), Q2.6 (COLLECTOR_#3_2): now also R4.2, U2.2 (-); no longer U2.3 (+)
- net at Q1.1 (COLLECTOR_DYE_#1), Q1.13 (BASE_#2), Q1.2 (COLLECTOR_#1): now also D2.3 (A)
- net at Q1.5 (COLLECTOR_#3_1), Q1.6 (COLLECTOR_#3_2): now also R3.2, U1.2 (-); no longer U1.3 (+)
Other:
- moved on the sheet: J2, J3, J5

Commit message: BNC Grounding
Connections:
- net GND: now also J1.1, J1.2
- no-connect marks 8 -> 6
Changed lines of the file:
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@@
+	)
+	(junction
+		(at 172.72 91.44)
+		(diameter 0)
+		(color 0 0 0 0)
 	)
 	(junction
@@
 	)
 	(junction
+		(at 148.59 95.25)
+		(diameter 0)
+		(color 0 0 0 0)
+	)
+	(junction
 		(at 76.2 134.62)
 		(diameter 0)
@@
 		(diameter 0)
 		(color 0 0 0 0)
-	)
-	(no_connect
-		(at 172.72 91.44)
 	)
 	(no_connect
@@
 	)
 	(no_connect
-		(at 172.72 88.9)
-	)
-	(no_connect
 		(at 92.71 87.63)
 	)
@@
 	(wire
 		(pts
-			(xy 148.59 27.94) (xy 148.59 135.89)
+			(xy 148.59 27.94) (xy 148.59 95.25)
 		)
 		(stroke
@@
 	(wire
 		(pts
+			(xy 172.72 88.9) (xy 172.72 91.44)
+		)
+		(stroke
+			(width 0)
+			(type default)
+		)
+	)
+	(wire
+		(pts
 			(xy 113.03 38.1) (xy 113.03 43.18)
 		)
@@
 	(wire
 		(pts
+			(xy 148.59 95.25) (xy 148.59 135.89)
+		)
+		(stroke
+			(width 0)
+			(type default)
+		)
+	)
+	(wire
+		(pts
+			(xy 148.59 95.25) (xy 172.72 95.25)
+		)
+		(stroke
+			(width 0)
+			(type default)
+		)
+	)
+	(wire
+		(pts
 			(xy 116.84 82.55) (xy 116.84 88.9)
 		)
@@
 		)
 		(stroke
+			(width 0)
+			(type default)
+		)
+	)
+	(wire
+		(pts
+			(xy 172.72 91.44) (xy 172.72 95.25)
+		)
+		(stroke

Commit message: Added Caps and Bias Change
Parts:
- added C1, C2: C_Polarized, Capacitor_THT:CP_Radial_D5.0mm_P2.50mm, symbol Device:C_Polarized
Connections:
- net +5V: now also D1.1 (K), D2.1 (K), C2.1
- net -5V: now also C1.1; no longer D1.1 (K), D2.1 (K)
- net GND: now also C1.2, C2.2

Commit message: Added caps to schematic
Parts:
- added C3, C4, C5, C6, C7, C8: C_Polarized, Capacitor_THT:CP_Radial_D5.0mm_P2.50mm, symbol Device:C_Polarized
Connections:
- net +5V: now also C3.1, C5.1, C7.1
- net -5V: now also C4.1, C6.1, C8.1
- net GND: now also C3.2, C4.2, C5.2, C6.2, C7.2, C8.2

Commit message: Changed the cap types
Parts:
- removed C3, C4, C5, C6, C7, C8: C_Polarized, Capacitor_THT:CP_Radial_D5.0mm_P2.50mm, symbol Device:C_Polarized
- added C10, C11, C12, C13, C14, C9: C, symbol Device:C
Connections:
- net +5V: now also C10.1, C11.1, C13.1
- net -5V: now also C12.2, C14.1, C9.2
- net GND: now also C10.2, C11.2, C12.1, C13.2, C14.2, C9.1

Commit message: Finalized the PCB Design
Parts:
- C1, C2: value C_Polarized -> 1u
- C10, C11, C12, C13, C14, C9: value C -> 100n; footprint (none) -> Capacitor_THT:C_Disc_D3.0mm_W1.6mm_P2.50mm
Changed lines of the file:
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@@
 			)
 		)
-		(property "Value" "C"
+		(property "Value" "100n"
 			(at 80.01 68.58 90)
 			(effects
@@
 			)
 		)
-		(property "Footprint" ""
+		(property "Footprint" "Capacitor_THT:C_Disc_D3.0mm_W1.6mm_P2.50mm"
 			(at 76.2 74.6252 0)
 			(effects
@@
 			)
 		)
-		(property "Value" "C_Polarized"
+		(property "Value" "1u"
 			(at 157.48 122.3009 0)
 			(effects
@@
 			)
 		)
-		(property "Value" "C_Polarized"
+		(property "Value" "1u"
 			(at 157.48 112.1409 0)
 			(effects
@@
 			)
 		)
-		(property "Value" "C"
+		(property "Value" "100n"
 			(at 146.05 109.2199 0)
 			(effects
@@
 			)
 		)
-		(property "Footprint" ""
+		(property "Footprint" "Capacitor_THT:C_Disc_D3.0mm_W1.6mm_P2.50mm"
 			(at 143.2052 111.76 0)
 			(effects
@@
 			)
 		)
-		(property "Value" "C"
+		(property "Value" "100n"
 			(at 66.04 83.8199 0)
 			(effects
@@
 			)
 		)
-		(property "Footprint" ""
+		(property "Footprint" "Capacitor_THT:C_Disc_D3.0mm_W1.6mm_P2.50mm"
 			(at 63.1952 86.36 0)
 			(effects
@@
 			)
 		)
-		(property "Value" "C"
+		(property "Value" "100n"
 			(at 137.16 74.9299 0)
 			(effects
@@
 			)
 		)
-		(property "Footprint" ""
+		(property "Footprint" "Capacitor_THT:C_Disc_D3.0mm_W1.6mm_P2.50mm"
 			(at 134.3152 77.47 0)
 			(effects
@@
 			)
 		)
-		(property "Value" "C"
+		(property "Value" "100n"
 			(at 46.99 106.6799 0)
 			(effects
@@
 			)
 		)
-		(property "Footprint" ""
+		(property "Footprint" "Capacitor_THT:C_Disc_D3.0mm_W1.6mm_P2.50mm"
 			(at 44.1452 109.22 0)
 			(effects
@@
 			)
 		)
-		(property "Value" "C"
+		(property "Value" "100n"
 			(at 64.77 92.71 90)
 			(effects
@@
 			)
 		)
-		(property "Footprint" ""
+		(property "Footprint" "Capacitor_THT:C_Disc_D3.0mm_W1.6mm_P2.50mm"
 			(at 60.96 98.7552 0)
 			(effects
